File: Schematic.kicad_sch (KiCad schematic)
At the start: 123 parts, among them Q1 NPN, SW1 SW_Push, SW2 SW_Push, SW4 SW_Push, SW5 DPDT, SW6 SW_Push, U1 74LS173, U10 74LS86, U11 74LS86, U12 74LS86, U13 74LS86, U14 74LS245, U15 7408, U16 7408, U17 7432, U18 74LS86, U19 74LS86, U2 74LS173, U20 74LS86, U21 74LS86, U22 7432, U23 ICM7555xB, U3 74LS245, U4 74LS173, U5 74LS173, U6 74LS86, U7 4008, U8 74LS86, U9 4008

Commit message: Added Schematic PDF
Parts:
- renumbered R333 to R330, R338 to R330, R332 to R330, R331 to R330, R336 to R330, R334 to R330, R337 to R330, R335 to R330
Changed lines of the file:
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@@
 		(in_pos_files yes)
 		(dnp no)
-		(property "Reference" "R333"
+		(property "Reference" "R330"
 			(at 115.57 234.95 90)
 			(show_name no)
@@
 			(project "Schematic"
 				(path "/91d74357-8ca4-4a58-80c6-cf56241b3e29"
-					(reference "R333")
+					(reference "R330")
 					(unit 1)
 				)
@@
 		(in_pos_files yes)
 		(dnp no)
-		(property "Reference" "R338"
+		(property "Reference" "R330"
 			(at 246.38 234.95 90)
 			(show_name no)
@@
 			(project "Schematic"
 				(path "/91d74357-8ca4-4a58-80c6-cf56241b3e29"
-					(reference "R338")
+					(reference "R330")
 					(unit 1)
 				)
@@
 		(in_pos_files yes)
 		(dnp no)
-		(property "Reference" "R332"
+		(property "Reference" "R330"
 			(at 90.17 234.95 90)
 			(show_name no)
@@
 			(project "Schematic"
 				(path "/91d74357-8ca4-4a58-80c6-cf56241b3e29"
-					(reference "R332")
+					(reference "R330")
 					(unit 1)
 				)
@@
 		(in_pos_files yes)
 		(dnp no)
-		(property "Reference" "R331"
+		(property "Reference" "R330"
 			(at 64.77 234.95 90)
 			(show_name no)
@@
 			(project "Schematic"
 				(path "/91d74357-8ca4-4a58-80c6-cf56241b3e29"
-					(reference "R331")
+					(reference "R330")
 					(unit 1)
 				)
@@
 		(in_pos_files yes)
 		(dnp no)
-		(property "Reference" "R336"
+		(property "Reference" "R330"
 			(at 193.04 234.95 90)
 			(show_name no)
@@
 			(project "Schematic"
 				(path "/91d74357-8ca4-4a58-80c6-cf56241b3e29"
-					(reference "R336")
+					(reference "R330")
 					(unit 1)
 				)
@@
 		(in_pos_files yes)
 		(dnp no)
-		(property "Reference" "R334"
+		(property "Reference" "R330"
 			(at 140.97 234.95 90)
 			(show_name no)
@@
 			(project "Schematic"
 				(path "/91d74357-8ca4-4a58-80c6-cf56241b3e29"
-					(reference "R334")
+					(reference "R330")
 					(unit 1)
 				)
@@
 		(in_pos_files yes)
 		(dnp no)
-		(property "Reference" "R337"
+		(property "Reference" "R330"
 			(at 219.71 234.95 90)
 			(show_name no)
@@
 			(project "Schematic"
 				(path "/91d74357-8ca4-4a58-80c6-cf56241b3e29"
-					(reference "R337")
+					(reference "R330")
 					(unit 1)
 				)
@@
 		(in_pos_files yes)
 		(dnp no)
-		(property "Reference" "R335"
+		(property "Reference" "R330"
 			(at 166.37 234.95 90)
 			(show_name no)
@@
 			(project "Schematic"
 				(path "/91d74357-8ca4-4a58-80c6-cf56241b3e29"
-					(reference "R335")
+					(reference "R330")
 					(unit 1)
 				)
